Commit message: WIP: batched solver collision + palm contact + routing + init push-out
Accumulated changes from multi-session iteration:
- Box collision primitives from MuJoCo Menagerie in LEAP URDF
- BoxCollisionModel in constrained_grasp_solver.py
- Hybrid collision: box corners for palm + PCA-filtered visual mesh for tips + visual mesh for body links
- Palm contact as 5th contact (nc=5) in wrench matrix
- Routing constraint (IF/MF/RF on palm side, TH opposite)
- Collision-free initialization with curl + push-out
- Full visual mesh verification post-solve
- Self-collision: inter-finger + palm-finger pairs
- Geometry-to-object surface loss (min SDF over ds collision points)
- Wrapping selection in Phase 1
- Feasibility filter with σ_min + opposing normals

Status: penetration mostly solved but tips still 16-24mm from surface.
Palm orientation sometimes wrong. Force closure weak.

Co-Authored-By: Claude Opus 4.6 (1M context) <noreply@anthropic.com>

File: models/leap_rh/leap.urdf (robot description, URDF)
Before this commit: robot onshape, 19 links, 18 joints
Links:
- link leap_rh_if_bs: geometry collision box size=0.014000 0.020000 0.004000; collision box size=0.014000 0.020000 0.004000
- link leap_rh_if_ds: geometry collision box size=0.014000 0.022000 0.004000; collision box size=0.014000 0.022000 0.004000
- link leap_rh_if_md: geometry collision box size=0.014000 0.020000 0.004000; collision box size=0.014000 0.020000 0.004000
- link leap_rh_if_px: geometry collision box size=0.034000 0.026000 0.022000; visual mesh filename=meshes_obj/pip.obj
- link leap_rh_mf_bs: geometry collision box size=0.014000 0.020000 0.004000; collision box size=0.014000 0.020000 0.004000
- link leap_rh_mf_ds: geometry collision box size=0.014000 0.022000 0.004000; collision box size=0.014000 0.022000 0.004000
- link leap_rh_mf_md: geometry collision box size=0.014000 0.020000 0.004000; collision box size=0.014000 0.020000 0.004000
- link leap_rh_mf_px: geometry collision box size=0.034000 0.026000 0.022000; visual mesh filename=meshes_obj/pip.obj
- link leap_rh_palm: geometry collision box size=0.004000 0.036000 0.034000; collision box size=0.010000 0.120000 0.020000
- link leap_rh_rf_bs: geometry collision box size=0.014000 0.020000 0.004000; collision box size=0.014000 0.020000 0.004000
- link leap_rh_rf_ds: geometry collision box size=0.014000 0.022000 0.004000; collision box size=0.014000 0.022000 0.004000
- link leap_rh_rf_md: geometry collision box size=0.014000 0.020000 0.004000; collision box size=0.014000 0.020000 0.004000
- link leap_rh_rf_px: geometry collision box size=0.034000 0.026000 0.022000; visual mesh filename=meshes_obj/pip.obj
- link leap_rh_th_bs: geometry collision box size=0.014000 0.004000 0.020000; collision box size=0.014000 0.004000 0.020000
- link leap_rh_th_ds: geometry collision box size=0.008000 0.024000 0.018000; collision box size=0.020000 0.004000 0.030000
- link leap_rh_th_mp: geometry collision box size=0.034000 0.026000 0.022000; visual mesh filename=meshes_obj/pip.obj
- link leap_rh_th_px: geometry collision box size=0.010000 0.024000 0.018000; collision box size=0.014000 0.020000 0.004000

Commit message: WIP: Full pipeline rework — tip coverage, link-level SC, 3-support+palm FC
Major changes from multi-session work:
- Box-grid collision (5mm URDF boxes) replaces sphere-based
- Visual mesh surface samples for ds (fingertip) links (covers 30mm gap)
- Link-level self-collision pairs (108 pairs vs 10 finger-level)
- 3 support fingers + palm FC (actuation excluded)
- CMC sector init for finger spreading
- Variant A/B/C optimization system (A = baseline soft penalty, best so far)
- Analytical box_box_sdf_batch (implemented but unused — too slow in loop)
- SC adjacency fix (palm↔bs excluded)
- Same-finger pairs excluded from SC

Known issues (pre-cleanup):
- ~920 lines dead Phase 0-2 code after early return
- Section B does NOT check ds links for collision (sfx_no_ds)
- Verification SC uses _col_data, optimizer uses _sc_data (inconsistent)
- No actuation area exclusion for support fingers
- Unused functions: compute_fc_proxy_loss, min_weight_gradient_batch, etc.

Co-Authored-By: Claude Opus 4.6 (1M context) <noreply@anthropic.com>

File: models/leap_rh/leap.urdf (robot description, URDF)
Before this commit: robot onshape, 19 links, 18 joints
Links:
- link leap_rh_mf_ds: geometry collision box size=0.014000 0.022000 0.004000; collision box size=0.014000 0.022000 0.004000
- link leap_rh_rf_ds: geometry collision box size=0.014000 0.022000 0.004000; collision box size=0.014000 0.022000 0.004000
